Commit message: fix: robot wheel origin

File: src/iot_robot_description/urdf/robot.urdf.xacro (robot description, xacro)
@@ -99,5 +99,5 @@
         </inertial>
         <visual>
-            <origin xyz="0.000053 0 0" rpy="0 0 0" />
+            <origin xyz="0.00534 0 0" rpy="0 0 0" />
             <geometry>
                 <mesh filename="package://iot_robot_description/meshes/wheel_link_left_visual.stl" />
@@ -118,5 +118,5 @@
         </inertial>
         <visual>
-            <origin xyz="0.000053 0 0" rpy="0 0 0" />
+            <origin xyz="0.00534 0 0" rpy="0 0 0" />
             <geometry>
                 <mesh filename="package://iot_robot_description/meshes/wheel_link_right_visual.stl" />

Commit message: feat: simulated ultrasonic sensors
Adds ultrasonic_left_link and ultrasonic_right_link frames to the description
and models each HC-SR04 as five MuJoCo rangefinder rays across its cone.
scan_to_range turns the resulting LaserScans into the sensor_msgs/Range
messages the STM32 bridge publishes on the real robot. The scene gains a wall
and a crate, outside the camera's view, for the sensors to see.

File: src/iot_robot_description/urdf/robot.urdf.xacro (robot description, xacro)
@@ -188,3 +188,18 @@
         <child link="camera_optical_frame" />
     </joint>
+    <!-- HC-SR04 ultrasonic sensors on the two front chamfers, turned 45° outwards. The origin
+         sits just in front of the transducer faces (their centre is 30 mm above base_link) and
+         x points along the beam, so sensor_msgs/Range readings are measured from this frame -->
+    <link name="ultrasonic_left_link" />
+    <joint name="ultrasonic_left_joint" type="fixed">
+        <origin xyz="0.144 0.114 0.030" rpy="0 0 ${pi/4}" />
+        <parent link="base_link" />
+        <child link="ultrasonic_left_link" />
+    </joint>
+    <link name="ultrasonic_right_link" />
+    <joint name="ultrasonic_right_joint" type="fixed">
+        <origin xyz="0.144 -0.114 0.030" rpy="0 0 ${-pi/4}" />
+        <parent link="base_link" />
+        <child link="ultrasonic_right_link" />
+    </joint>
 </robot>

File: src/iot_robot_mujoco/urdf/iot_robot_sim.urdf.xacro (robot description, xacro)
@@ -11,4 +11,6 @@
             <param name="headless">$(arg headless)</param>
             <param name="camera_publish_rate">15.0</param>
+            <!-- The STM32 reports both ultrasonic sensors at about 15 Hz -->
+            <param name="lidar_publish_rate">15.0</param>
         </hardware>
         <joint name="wheel_joint_left">
@@ -39,4 +41,26 @@
             <param name="depth_topic">/camera/depth</param>
         </sensor>
+        <!-- Ultrasonic sensors. Each name matches the ultrasonic_*-N rangefinders created by the
+         <lidar> tags in mujoco_inputs.xml, and the angles must match those tags. The plugin
+         publishes a 5-ray LaserScan; scan_to_range turns it into the sensor_msgs/Range that
+         the STM32 bridge publishes on the real robot -->
+        <sensor name="ultrasonic_left">
+            <param name="frame_name">ultrasonic_left_link</param>
+            <param name="min_angle">-0.13</param>
+            <param name="max_angle">0.13</param>
+            <param name="angle_increment">0.065</param>
+            <param name="range_min">0.02</param>
+            <param name="range_max">4.0</param>
+            <param name="laserscan_topic">/sim/ultrasonic/left/scan</param>
+        </sensor>
+        <sensor name="ultrasonic_right">
+            <param name="frame_name">ultrasonic_right_link</param>
+            <param name="min_angle">-0.13</param>
+            <param name="max_angle">0.13</param>
+            <param name="angle_increment">0.065</param>
+            <param name="range_min">0.02</param>
+            <param name="range_max">4.0</param>
+            <param name="laserscan_topic">/sim/ultrasonic/right/scan</param>
+        </sensor>
     </ros2_control>
 </robot>

Commit message: feat: LSM9DS1 IMU on the Raspberry Pi's I2C bus
- lsm9ds1 driver (smbus2) with datasheet scaling to SI units, the
  magnetometer axes mapped into the accelerometer/gyroscope frame and an
  optional gyroscope bias estimate at start-up
- lsm9ds1_node publishes /imu/data_raw and /imu/mag and retries when the
  sensor is missing instead of exiting
- imu.launch.py runs it with imu_filter_madgwick (/imu/data, magnetometer
  off by default because of the motors nearby)
- imu_link in the description URDF, pose still to be measured
- install.sh enables I2C with raspi-config, installs i2c-tools and adds
  the user to the i2c group

File: src/iot_robot_description/urdf/robot.urdf.xacro (robot description, xacro)
@@ -203,3 +203,17 @@
         <child link="ultrasonic_right_link" />
     </joint>
+    <!-- LSM9DS1 IMU. imu_link has the magnetometer's axes, the right-handed set that
+         lsm9ds1_node reports in (iot_robot_drivers/lsm9ds1.py): seen from above with the
+         chip's pin 1 dot at the top left, x points left, y down the page and z up out of it.
+         PLACEHOLDER POSE: measure where the chip sits relative to base_link and how it is
+         turned, then set xyz and rpy. To check the rotation, stand the robot level: the
+         imu_link axis pointing up reads about +9.8 m/s^2 in imu/data_raw, and turning the
+         robot to the left gives a positive angular velocity about that same axis. With
+         rpy 0 0 0 both must show on z -->
+    <link name="imu_link" />
+    <joint name="imu_joint" type="fixed">
+        <origin xyz="0 0 0.05" rpy="0 0 0" />
+        <parent link="base_link" />
+        <child link="imu_link" />
+    </joint>
 </robot>
